Commit message: Add foot contact spheres + model provenance (LICENSE/SOURCE) for K1/R1/H1-2/T1
Co-Authored-By: Claude Fable 5 <noreply@anthropic.com>

File: src/holosoma_retargeting/holosoma_retargeting/models/h1_2/h1_2_27dof.urdf (robot description, URDF)
Before this commit: robot h1_2, 32 links, 31 joints
Links:
- added link left_ankle_roll_sphere_1_link, mass 0.001; collision sphere radius=0.005; visual sphere radius=0.005
- added link left_ankle_roll_sphere_2_link, mass 0.001; collision sphere radius=0.005; visual sphere radius=0.005
- added link left_ankle_roll_sphere_3_link, mass 0.001; collision sphere radius=0.005; visual sphere radius=0.005
- added link left_ankle_roll_sphere_4_link, mass 0.001; collision sphere radius=0.005; visual sphere radius=0.005
- added link left_ankle_roll_sphere_5_link, mass 0.001; collision sphere radius=0.005; visual sphere radius=0.005
- added link right_ankle_roll_sphere_1_link, mass 0.001; collision sphere radius=0.005; visual sphere radius=0.005
- added link right_ankle_roll_sphere_2_link, mass 0.001; collision sphere radius=0.005; visual sphere radius=0.005
- added link right_ankle_roll_sphere_3_link, mass 0.001; collision sphere radius=0.005; visual sphere radius=0.005
- added link right_ankle_roll_sphere_4_link, mass 0.001; collision sphere radius=0.005; visual sphere radius=0.005
- added link right_ankle_roll_sphere_5_link, mass 0.001; collision sphere radius=0.005; visual sphere radius=0.005
Joints:
- added joint left_ankle_roll_sphere_1_joint: type fixed, parent left_ankle_roll_link, child left_ankle_roll_sphere_1_link, origin xyz=-0.075 0.028 -0.04 rpy=0 0 0
- added joint left_ankle_roll_sphere_2_joint: type fixed, parent left_ankle_roll_link, child left_ankle_roll_sphere_2_link, origin xyz=-0.075 -0.028 -0.04 rpy=0 0 0
- added joint left_ankle_roll_sphere_3_joint: type fixed, parent left_ankle_roll_link, child left_ankle_roll_sphere_3_link, origin xyz=0.155 0.034 -0.04 rpy=0 0 0
- added joint left_ankle_roll_sphere_4_joint: type fixed, parent left_ankle_roll_link, child left_ankle_roll_sphere_4_link, origin xyz=0.155 -0.034 -0.04 rpy=0 0 0
- added joint left_ankle_roll_sphere_5_joint: type fixed, parent left_ankle_roll_link, child left_ankle_roll_sphere_5_link, origin xyz=0.17 0 -0.04 rpy=0 0 0
- added joint right_ankle_roll_sphere_1_joint: type fixed, parent right_ankle_roll_link, child right_ankle_roll_sphere_1_link, origin xyz=-0.075 0.028 -0.04 rpy=0 0 0
- added joint right_ankle_roll_sphere_2_joint: type fixed, parent right_ankle_roll_link, child right_ankle_roll_sphere_2_link, origin xyz=-0.075 -0.028 -0.04 rpy=0 0 0
- added joint right_ankle_roll_sphere_3_joint: type fixed, parent right_ankle_roll_link, child right_ankle_roll_sphere_3_link, origin xyz=0.155 0.034 -0.04 rpy=0 0 0
- added joint right_ankle_roll_sphere_4_joint: type fixed, parent right_ankle_roll_link, child right_ankle_roll_sphere_4_link, origin xyz=0.155 -0.034 -0.04 rpy=0 0 0
- added joint right_ankle_roll_sphere_5_joint: type fixed, parent right_ankle_roll_link, child right_ankle_roll_sphere_5_link, origin xyz=0.17 0 -0.04 rpy=0 0 0

File: src/holosoma_retargeting/holosoma_retargeting/models/k1/k1_22dof.urdf (robot description, URDF)
Before this commit: robot K1, 23 links, 22 joints
Links:
- added link left_foot_sphere_1_link, mass 0.001; collision sphere radius=0.005; visual sphere radius=0.005
- added link left_foot_sphere_2_link, mass 0.001; collision sphere radius=0.005; visual sphere radius=0.005
- added link left_foot_sphere_3_link, mass 0.001; collision sphere radius=0.005; visual sphere radius=0.005
- added link left_foot_sphere_4_link, mass 0.001; collision sphere radius=0.005; visual sphere radius=0.005
- added link left_foot_sphere_5_link, mass 0.001; collision sphere radius=0.005; visual sphere radius=0.005
- added link right_foot_sphere_1_link, mass 0.001; collision sphere radius=0.005; visual sphere radius=0.005
- added link right_foot_sphere_2_link, mass 0.001; collision sphere radius=0.005; visual sphere radius=0.005
- added link right_foot_sphere_3_link, mass 0.001; collision sphere radius=0.005; visual sphere radius=0.005
- added link right_foot_sphere_4_link, mass 0.001; collision sphere radius=0.005; visual sphere radius=0.005
- added link right_foot_sphere_5_link, mass 0.001; collision sphere radius=0.005; visual sphere radius=0.005
Joints:
- added joint left_foot_sphere_1_joint: type fixed, parent left_foot_link, child left_foot_sphere_1_link, origin xyz=-0.055 0.022 -0.035 rpy=0 0 0
- added joint left_foot_sphere_2_joint: type fixed, parent left_foot_link, child left_foot_sphere_2_link, origin xyz=-0.055 -0.022 -0.035 rpy=0 0 0
- added joint left_foot_sphere_3_joint: type fixed, parent left_foot_link, child left_foot_sphere_3_link, origin xyz=0.095 0.028 -0.035 rpy=0 0 0
- added joint left_foot_sphere_4_joint: type fixed, parent left_foot_link, child left_foot_sphere_4_link, origin xyz=0.095 -0.028 -0.035 rpy=0 0 0
- added joint left_foot_sphere_5_joint: type fixed, parent left_foot_link, child left_foot_sphere_5_link, origin xyz=0.11 0 -0.035 rpy=0 0 0
- added joint right_foot_sphere_1_joint: type fixed, parent right_foot_link, child right_foot_sphere_1_link, origin xyz=-0.055 0.022 -0.035 rpy=0 0 0
- added joint right_foot_sphere_2_joint: type fixed, parent right_foot_link, child right_foot_sphere_2_link, origin xyz=-0.055 -0.022 -0.035 rpy=0 0 0
- added joint right_foot_sphere_3_joint: type fixed, parent right_foot_link, child right_foot_sphere_3_link, origin xyz=0.095 0.028 -0.035 rpy=0 0 0
- added joint right_foot_sphere_4_joint: type fixed, parent right_foot_link, child right_foot_sphere_4_link, origin xyz=0.095 -0.028 -0.035 rpy=0 0 0
- added joint right_foot_sphere_5_joint: type fixed, parent right_foot_link, child right_foot_sphere_5_link, origin xyz=0.11 0 -0.035 rpy=0 0 0

File: src/holosoma_retargeting/holosoma_retargeting/models/r1/r1_26dof.urdf (robot description, URDF)
Before this commit: robot R1, 40 links, 39 joints
Links:
- added link left_ankle_roll_sphere_1_link, mass 0.001; collision sphere radius=0.005; visual sphere radius=0.005
- added link left_ankle_roll_sphere_2_link, mass 0.001; collision sphere radius=0.005; visual sphere radius=0.005
- added link left_ankle_roll_sphere_3_link, mass 0.001; collision sphere radius=0.005; visual sphere radius=0.005
- added link left_ankle_roll_sphere_4_link, mass 0.001; collision sphere radius=0.005; visual sphere radius=0.005
- added link left_ankle_roll_sphere_5_link, mass 0.001; collision sphere radius=0.005; visual sphere radius=0.005
- added link right_ankle_roll_sphere_1_link, mass 0.001; collision sphere radius=0.005; visual sphere radius=0.005
- added link right_ankle_roll_sphere_2_link, mass 0.001; collision sphere radius=0.005; visual sphere radius=0.005
- added link right_ankle_roll_sphere_3_link, mass 0.001; collision sphere radius=0.005; visual sphere radius=0.005
- added link right_ankle_roll_sphere_4_link, mass 0.001; collision sphere radius=0.005; visual sphere radius=0.005
- added link right_ankle_roll_sphere_5_link, mass 0.001; collision sphere radius=0.005; visual sphere radius=0.005
Joints:
- added joint left_ankle_roll_sphere_1_joint: type fixed, parent left_ankle_roll_link, child left_ankle_roll_sphere_1_link, origin xyz=-0.045 0.022 -0.05 rpy=0 0 0
- added joint left_ankle_roll_sphere_2_joint: type fixed, parent left_ankle_roll_link, child left_ankle_roll_sphere_2_link, origin xyz=-0.045 -0.022 -0.05 rpy=0 0 0
- added joint left_ankle_roll_sphere_3_joint: type fixed, parent left_ankle_roll_link, child left_ankle_roll_sphere_3_link, origin xyz=0.115 0.028 -0.05 rpy=0 0 0
- added joint left_ankle_roll_sphere_4_joint: type fixed, parent left_ankle_roll_link, child left_ankle_roll_sphere_4_link, origin xyz=0.115 -0.028 -0.05 rpy=0 0 0
- added joint left_ankle_roll_sphere_5_joint: type fixed, parent left_ankle_roll_link, child left_ankle_roll_sphere_5_link, origin xyz=0.13 0 -0.05 rpy=0 0 0
- added joint right_ankle_roll_sphere_1_joint: type fixed, parent right_ankle_roll_link, child right_ankle_roll_sphere_1_link, origin xyz=-0.045 0.022 -0.05 rpy=0 0 0
- added joint right_ankle_roll_sphere_2_joint: type fixed, parent right_ankle_roll_link, child right_ankle_roll_sphere_2_link, origin xyz=-0.045 -0.022 -0.05 rpy=0 0 0
- added joint right_ankle_roll_sphere_3_joint: type fixed, parent right_ankle_roll_link, child right_ankle_roll_sphere_3_link, origin xyz=0.115 0.028 -0.05 rpy=0 0 0
- added joint right_ankle_roll_sphere_4_joint: type fixed, parent right_ankle_roll_link, child right_ankle_roll_sphere_4_link, origin xyz=0.115 -0.028 -0.05 rpy=0 0 0
- added joint right_ankle_roll_sphere_5_joint: type fixed, parent right_ankle_roll_link, child right_ankle_roll_sphere_5_link, origin xyz=0.13 0 -0.05 rpy=0 0 0
