Commit message: Add R1 asset / Add extension for the arm part so that it retargets better for R1 / G1

File: src/holosoma_retargeting/holosoma_retargeting/models/r1/r1_24dof.urdf (robot description, URDF)
Before this commit: robot R1, 50 links, 49 joints
Links:
- added link left_hand_sphere_link, mass 0.001; visual sphere radius=0.005
- added link right_hand_sphere_link, mass 0.001; visual sphere radius=0.005
Joints:
- added joint left_hand_sphere_joint: type fixed, parent left_wrist_roll_link, child left_hand_sphere_link, origin xyz=0.1 0 0 rpy=0 0 0
- added joint right_hand_sphere_joint: type fixed, parent right_wrist_roll_link, child right_hand_sphere_link, origin xyz=0.1 0 0 rpy=0 0 0
